Commit message: fix(etrike): refine tuktuk body silhouette

File: autoware/src/our_packages/etrike_vehicle_description/urdf/vehicle.xacro (robot description, xacro)
@@ -18,7 +18,8 @@
   <xacro:property name="overall_height" value="1.700"/>
   <xacro:property name="ground_clearance" value="0.170"/>
-  <!-- Estimated split; replace after measuring the physical vehicle. -->
-  <xacro:property name="front_overhang" value="0.350"/>
-  <xacro:property name="rear_overhang" value="0.285"/>
+  <!-- Visual-envelope split: front tire edge to rear body panel. Measure the
+       physical vehicle before footprint-critical deployment. -->
+  <xacro:property name="front_overhang" value="0.203"/>
+  <xacro:property name="rear_overhang" value="0.432"/>
   <material name="body_blue"><color rgba="0.035 0.235 0.510 1.0"/></material>
   <material name="tire_black"><color rgba="0.025 0.025 0.030 1.0"/></material>

Commit message: fix(etrike): refine body profile and dimensions

File: autoware/src/our_packages/etrike_vehicle_description/urdf/vehicle.xacro (robot description, xacro)
@@ -48,5 +48,5 @@
     </collision>
     <collision name="lower_body_collision">
-      <origin xyz="0.583 0 0.550" rpy="0 0 0"/>
+      <origin xyz="0.583 0 0.555" rpy="0 0 0"/>
       <geometry><box size="1.735 0.900 0.550"/></geometry>
     </collision>
@@ -120,10 +120,10 @@
   <link name="front_steering_link">
     <inertial>
-      <origin xyz="-0.030 0 0.180" rpy="0 0 0"/>
+      <origin xyz="-0.030 0 0.383" rpy="0 0 0"/>
       <mass value="1.0"/>
       <inertia ixx="0.0078" ixy="0" ixz="0" iyy="0.0078" iyz="0" izz="0.0006"/>
     </inertial>
     <collision name="steering_carrier_collision">
-      <origin xyz="-0.030 0 0.180" rpy="0 0 0"/>
+      <origin xyz="-0.030 0 0.383" rpy="0 0 0"/>
       <geometry><box size="0.060 0.060 0.360"/></geometry>
     </collision>

Commit message: feat(etrike): add simplified Hesai XT32M2X 3D LiDAR cylinder at top center of flat roof deck with ROS 2 lidar_link

File: autoware/src/our_packages/etrike_vehicle_description/urdf/vehicle.xacro (robot description, xacro)
@@ -161,3 +161,33 @@
     <dynamics damping="0.05" friction="0.02"/>
   </joint>
+  <!-- Hesai XT32M2X 3D LiDAR Link (Autoware / ROS 2) -->
+  <xacro:property name="lidar_x" value="0.575"/>
+  <xacro:property name="lidar_y" value="0.000"/>
+  <xacro:property name="lidar_roof_z" value="1.700"/>
+  <xacro:property name="lidar_optical_height" value="0.0464"/>
+  <xacro:property name="lidar_total_height" value="0.075"/>
+  <xacro:property name="lidar_radius" value="0.0465"/>
+  <material name="lidar_dark_grey"><color rgba="0.15 0.15 0.18 1.0"/></material>
+  <link name="lidar_link">
+    <inertial>
+      <origin xyz="0 0 0" rpy="0 0 0"/>
+      <mass value="0.490"/>
+      <inertia ixx="0.00049" ixy="0" ixz="0" iyy="0.00049" iyz="0" izz="0.00053"/>
+    </inertial>
+    <visual name="hesai_xt32m2x_visual">
+      <origin xyz="0 0 ${-lidar_optical_height + (lidar_total_height / 2.0)}" rpy="0 0 0"/>
+      <geometry><cylinder radius="${lidar_radius}" length="${lidar_total_height}"/></geometry>
+      <material name="lidar_dark_grey"/>
+    </visual>
+    <collision name="hesai_xt32m2x_collision">
+      <origin xyz="0 0 ${-lidar_optical_height + (lidar_total_height / 2.0)}" rpy="0 0 0"/>
+      <geometry><cylinder radius="${lidar_radius}" length="${lidar_total_height}"/></geometry>
+    </collision>
+  </link>
+  <joint name="lidar_joint" type="fixed">
+    <parent link="base_link"/>
+    <child link="lidar_link"/>
+    <!-- Sensor frame origin matches Hesai optical measurement origin (+46.4mm above roof) -->
+    <origin xyz="${lidar_x} ${lidar_y} ${lidar_roof_z + lidar_optical_height}" rpy="0 0 0"/>
+  </joint>
 </robot>

Commit message: docs: update documentation with build fixes, test results, and PandarView2 info
- SETUP_COMPLETE.md: Update directory structure, mark completed items
- RT_SYS_COMPATIBILITY.md: Add build status and Humble fixes
- TEST_PLAN.md: Add test results summary
- PANDARVIEW2.md: New document for PandarView2 (x86_64 only)

File: autoware/src/our_packages/etrike_vehicle_description/urdf/vehicle.xacro (robot description, xacro)
@@ -39,5 +39,5 @@
       <origin xyz="0 0 0" rpy="0 0 0"/>
       <geometry>
-        <mesh filename="package://etrike_vehicle_description/meshes/etrike_body.stl" scale="1 1 1"/>
+        <mesh filename="package://etrike_vehicle_description/meshes/etrike_body_binary.stl" scale="1 1 1"/>
       </geometry>
       <material name="body_blue"/>

Commit message: fix(pipeline): improve stop_all with clean container restart and browser cleanup

File: autoware/src/our_packages/etrike_vehicle_description/urdf/vehicle.xacro (robot description, xacro)
@@ -13,5 +13,5 @@
   <xacro:property name="wheel_radius" value="0.203"/>
   <xacro:property name="wheel_width" value="0.102"/>
-  <xacro:property name="max_steer_angle" value="0.747"/>
+  <xacro:property name="max_steer_angle" value="0.314"/>
   <xacro:property name="overall_length" value="2.635"/>
   <xacro:property name="overall_width" value="1.300"/>
