Commit message: fix(vehicle): make planning-sim URDF render full tuktuk model
The planning simulator (simple_planning_simulator) never publishes
/joint_states, so robot_state_publisher could not emit TF for the
etrike URDF's movable wheel/steering joints (continuous/revolute).
This left the wheel links without a transform, causing RViz's
RobotModel to error and the 3 wheels to not render.

- etrike_vehicle_description/urdf/vehicle.xacro: change the two rear
  wheel, front steering, and front wheel joints from continuous/revolute
  to fixed, matching the upstream single-mesh planning-sim convention
  (e.g. sample_vehicle). RSP now publishes all frames statically.
- etrike_kinect2/urdf/kinect_v2.xacro and etrike_sensor_kit_description/
  urdf/sensors.xacro: remove colons from XML comment text that broke
  launch's YAML parsing of the generated robot_description param.

- Also fixes a launch failure where colon-containing comments in the
  URDF were parsed as YAML and aborted the planning_simulator launch.

File: autoware/src/our_packages/etrike_kinect2/urdf/kinect_v2.xacro (robot description, xacro)
@@ -3,14 +3,14 @@
   <!--
     Microsoft Kinect v2 (Kinect One) sensor frames.
-    Physical dimensions (approximate):
-      Body: 249mm x 66mm x 67mm (W x H x D)
-      Depth range: 0.5 – 4.5 m
-      RGB: 1920x1080, Depth/IR: 512x424
-    Frame convention:
-      - Kinect sensor frame: X-right, Y-down, Z-forward (into scene)
-      - Optical frame: X-right, Y-down, Z-forward
+    Physical dimensions (approximate)
+      Body 249mm x 66mm x 67mm (W x H x D)
+      Depth range 0.5 - 4.5 m
+      RGB 1920x1080, Depth/IR 512x424
+    Frame convention
+      - Kinect sensor frame X-right, Y-down, Z-forward (into scene)
+      - Optical frame X-right, Y-down, Z-forward
         (same as sensor frame for Kinect v2)
-    Two instances: front (facing forward) and rear (facing backward).
-    Extrinsic poses are placeholders — calibrate after physical mounting.
+    Two instances front (facing forward) and rear (facing backward).
+    Extrinsic poses are placeholders - calibrate after physical mounting.
   -->
   <xacro:macro name="kinect_v2_macro" params="name parent x y z roll pitch yaw">

File: autoware/src/our_packages/etrike_sensor_kit_description/urdf/sensors.xacro (robot description, xacro)
@@ -7,5 +7,5 @@
   <!-- Kinect v2 cameras -->
   <xacro:include filename="$(find etrike_kinect2)/urdf/kinect_v2.xacro"/>
-  <!-- FRONT Kinect: windshield area, facing forward -->
+  <!-- FRONT Kinect - windshield area, facing forward -->
   <xacro:kinect_v2_macro
     name="kinect_front"
@@ -18,5 +18,5 @@
     yaw="${calibration['base_link']['kinect_front']['yaw']}"
   />
-  <!-- REAR Kinect: behind cabin, facing backward -->
+  <!-- REAR Kinect - behind cabin, facing backward -->
   <xacro:kinect_v2_macro
     name="kinect_rear"

File: autoware/src/our_packages/etrike_vehicle_description/urdf/vehicle.xacro (robot description, xacro)
@@ -85,11 +85,8 @@
     </collision>
   </link>
-  <joint name="rear_left_wheel_joint" type="continuous">
+  <joint name="rear_left_wheel_joint" type="fixed">
     <parent link="base_link"/>
     <child link="rear_left_wheel_link"/>
     <origin xyz="0 ${half_rear_track} ${wheel_radius}" rpy="0 0 0"/>
-    <axis xyz="0 1 0"/>
-    <limit effort="120.0" velocity="45.0"/>
-    <dynamics damping="0.05" friction="0.02"/>
   </joint>
   <link name="rear_right_wheel_link">
@@ -109,11 +106,8 @@
     </collision>
   </link>
-  <joint name="rear_right_wheel_joint" type="continuous">
+  <joint name="rear_right_wheel_joint" type="fixed">
     <parent link="base_link"/>
     <child link="rear_right_wheel_link"/>
     <origin xyz="0 -${half_rear_track} ${wheel_radius}" rpy="0 0 0"/>
-    <axis xyz="0 1 0"/>
-    <limit effort="120.0" velocity="45.0"/>
-    <dynamics damping="0.05" friction="0.02"/>
   </joint>
   <!-- Steering knuckle is at the documented front-wheel center. -->
@@ -129,11 +123,8 @@
     </collision>
   </link>
-  <joint name="front_steering_joint" type="revolute">
+  <joint name="front_steering_joint" type="fixed">
     <parent link="base_link"/>
     <child link="front_steering_link"/>
     <origin xyz="${wheel_base} 0 ${wheel_radius}" rpy="0 0 0"/>
-    <axis xyz="0 0 1"/>
-    <limit lower="-${max_steer_angle}" upper="${max_steer_angle}" effort="200.0" velocity="1.5"/>
-    <dynamics damping="2.0" friction="1.0"/>
   </joint>
   <link name="front_wheel_link">
@@ -153,11 +144,8 @@
     </collision>
   </link>
-  <joint name="front_wheel_joint" type="continuous">
+  <joint name="front_wheel_joint" type="fixed">
     <parent link="front_steering_link"/>
     <child link="front_wheel_link"/>
     <origin xyz="0 0 0" rpy="0 0 0"/>
-    <axis xyz="0 1 0"/>
-    <limit effort="120.0" velocity="45.0"/>
-    <dynamics damping="0.05" friction="0.02"/>
   </joint>
   <!-- Hesai XT32M2X 3D LiDAR Link (Autoware / ROS 2) -->

Commit message: fix(stack): integrate Hesai/Kinect2 sensing, ROS2 bridge, and open-etrike pipeline

File: autoware/src/our_packages/etrike_kinect2/urdf/kinect_v2.xacro (robot description, xacro)
@@ -15,14 +15,14 @@
   -->
   <xacro:macro name="kinect_v2_macro" params="name parent x y z roll pitch yaw">
-    <!-- Sensor body link -->
+    <!-- Sensor body link (ROS body convention: +X forward, +Y left, +Z up) -->
     <link name="${name}_link">
       <visual name="body">
         <origin xyz="0 0 0.0335" rpy="0 0 0"/>
-        <geometry><box size="0.249 0.066 0.067"/></geometry>
+        <geometry><box size="0.067 0.249 0.066"/></geometry>
         <material name="kinect_dark"><color rgba="0.1 0.1 0.12 1.0"/></material>
       </visual>
       <collision>
         <origin xyz="0 0 0.0335" rpy="0 0 0"/>
-        <geometry><box size="0.249 0.066 0.067"/></geometry>
+        <geometry><box size="0.067 0.249 0.066"/></geometry>
       </collision>
     </link>
@@ -32,24 +32,24 @@
       <origin xyz="${x} ${y} ${z}" rpy="${roll} ${pitch} ${yaw}"/>
     </joint>
-    <!-- RGB optical frame (same as sensor frame for Kinect v2) -->
+    <!-- RGB optical frame (REP-103 optical convention: +Z forward, +X right, +Y down) -->
     <link name="${name}_rgb_optical_frame"/>
     <joint name="${name}_rgb_optical_joint" type="fixed">
       <parent link="${name}_link"/>
       <child link="${name}_rgb_optical_frame"/>
-      <origin xyz="0 0 0" rpy="0 0 0"/>
+      <origin xyz="0 0 0" rpy="-1.57079632679 0 -1.57079632679"/>
     </joint>
-    <!-- Depth/IR optical frame -->
+    <!-- Depth/IR optical frame (REP-103 optical convention: +Z forward, +X right, +Y down) -->
     <link name="${name}_depth_optical_frame"/>
     <joint name="${name}_depth_optical_joint" type="fixed">
       <parent link="${name}_link"/>
       <child link="${name}_depth_optical_frame"/>
-      <origin xyz="0 0 0" rpy="0 0 0"/>
+      <origin xyz="0 0 0" rpy="-1.57079632679 0 -1.57079632679"/>
     </joint>
-    <!-- IR optical frame -->
+    <!-- IR optical frame (REP-103 optical convention: +Z forward, +X right, +Y down) -->
     <link name="${name}_ir_optical_frame"/>
     <joint name="${name}_ir_optical_joint" type="fixed">
       <parent link="${name}_link"/>
       <child link="${name}_ir_optical_frame"/>
-      <origin xyz="0 0 0" rpy="0 0 0"/>
+      <origin xyz="0 0 0" rpy="-1.57079632679 0 -1.57079632679"/>
     </joint>
   </xacro:macro>

File: autoware/src/our_packages/etrike_vehicle_description/urdf/vehicle.xacro (robot description, xacro)
@@ -179,3 +179,10 @@
     <origin xyz="${lidar_x} ${lidar_y} ${lidar_roof_z + lidar_optical_height}" rpy="0 0 0"/>
   </joint>
+  <!-- IMU frame (co-located with base_link until dedicated IMU mount is calibrated) -->
+  <link name="imu_link"/>
+  <joint name="imu_joint" type="fixed">
+    <parent link="base_link"/>
+    <child link="imu_link"/>
+    <origin xyz="0 0 0" rpy="0 0 0"/>
+  </joint>
 </robot>
